File: hardware/electronics/PCBs/Trackpoint_KiCad/Buttons.kicad_sch (KiCad schematic)
At the start: 4 parts, among them SW2 D2LS-21, SW4 D2LS-21, SW6 D2LS-21, SW8 D2LS-21

Commit message: Update all components to jlcpcb compatible
Parts:
- renumbered SW2 to BTN.SW.2, SW4 to BTN.SW.4, SW6 to BTN.SW.6, SW8 to BTN.SW.8
Changed lines of the file:
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@@
 		(in_pos_files yes)
 		(dnp no)
-		(property "Reference" "SW4"
+		(property "Reference" "BTN.SW.4"
 			(at 172.466 74.93 90)
 			(show_name no)
@@
 			(project "Trackpoint"
 				(path "/f80cdd06-fe18-4f08-ad78-5d64af2b92b5/7f0b0dd4-adcc-4917-b582-7b19e68204af"
-					(reference "SW4")
+					(reference "BTN.SW.4")
 					(unit 1)
 				)
@@
 		(in_pos_files yes)
 		(dnp no)
-		(property "Reference" "SW6"
+		(property "Reference" "BTN.SW.6"
 			(at 172.466 115.57 90)
 			(show_name no)
@@
 			(project "Trackpoint"
 				(path "/f80cdd06-fe18-4f08-ad78-5d64af2b92b5/7f0b0dd4-adcc-4917-b582-7b19e68204af"
-					(reference "SW6")
+					(reference "BTN.SW.6")
 					(unit 1)
 				)
@@
 		(in_pos_files yes)
 		(dnp no)
-		(property "Reference" "SW2"
+		(property "Reference" "BTN.SW.2"
 			(at 106.426 74.93 90)
 			(show_name no)
@@
 			(project "Trackpoint"
 				(path "/f80cdd06-fe18-4f08-ad78-5d64af2b92b5/7f0b0dd4-adcc-4917-b582-7b19e68204af"
-					(reference "SW2")
+					(reference "BTN.SW.2")
 					(unit 1)
 				)
@@
 		(in_pos_files yes)
 		(dnp no)
-		(property "Reference" "SW8"
+		(property "Reference" "BTN.SW.8"
 			(at 106.426 115.57 90)
 			(show_name no)
@@
 			(project "Trackpoint"
 				(path "/f80cdd06-fe18-4f08-ad78-5d64af2b92b5/7f0b0dd4-adcc-4917-b582-7b19e68204af"
-					(reference "SW8")
+					(reference "BTN.SW.8")
 					(unit 1)
 				)
