File: hardware/electronics/PCBs/Trackpoint_KiCad/Connectors.kicad_sch (KiCad schematic)
At the start: 8 parts, among them J3 DX07S016JA1R1500

Commit message: Update all components to jlcpcb compatible
Parts:
- USB.Ra.1: renamed from Ra1; JLCPCB Part # (none) -> C17902; Manufacturer (none) -> UNI-ROYAL; Manufacturer Part # (none) -> 1206W4F1002T5E
- renumbered FB1 to USB.FB.1, FB2 to USB.FB.2, FB3 to USB.FB.3, J3 to USB.J.3, R6 to USB.R.6, R7 to USB.R.7, Z1 to USB.Z.1
Changed lines of the file:
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@@
 		(in_pos_files yes)
 		(dnp no)
-		(property "Reference" "FB2"
+		(property "Reference" "USB.FB.2"
 			(at 198.12 91.44 90)
 			(show_name no)
@@
 			(project "Trackpoint"
 				(path "/f80cdd06-fe18-4f08-ad78-5d64af2b92b5/a056f087-e621-494b-bb8a-f53c663bfa45"
-					(reference "FB2")
+					(reference "USB.FB.2")
 					(unit 1)
 				)
@@
 		(in_pos_files yes)
 		(dnp no)
-		(property "Reference" "Ra1"
+		(property "Reference" "USB.Ra.1"
 			(at 122.682 101.346 0)
 			(show_name no)
@@
 		(property "ALTIUM_VALUE" "10k 1%"
 			(at 122.682 106.426 0)
+			(show_name no)
+			(do_not_autoplace no)
+			(effects
+				(font
+					(size 1.27 1.27)
+				)
+				(justify right bottom)
+			)
+		)
+		(property "JLCPCB Part #" "C17902"
+			(at 122.682 106.426 0)
+			(hide yes)
+			(show_name no)
+			(do_not_autoplace no)
+			(effects
+				(font
+					(size 1.27 1.27)
+				)
+				(justify right bottom)
+			)
+		)
+		(property "Manufacturer" "UNI-ROYAL"
+			(at 122.682 106.426 0)
+			(hide yes)
+			(show_name no)
+			(do_not_autoplace no)
+			(effects
+				(font
+					(size 1.27 1.27)
+				)
+				(justify right bottom)
+			)
+		)
+		(property "Manufacturer Part #" "1206W4F1002T5E"
+			(at 122.682 106.426 0)
+			(hide yes)
 			(show_name no)
 			(do_not_autoplace no)
@@
 			(project "Trackpoint"
 				(path "/f80cdd06-fe18-4f08-ad78-5d64af2b92b5/a056f087-e621-494b-bb8a-f53c663bfa45"
-					(reference "Ra1")
+					(reference "USB.Ra.1")
 					(unit 2)
 				)
@@
 		(in_pos_files yes)
 		(dnp no)
-		(property "Reference" "Ra1"
+		(property "Reference" "USB.Ra.1"
 			(at 89.662 101.346 0)
 			(show_name no)
@@
 		(property "ALTIUM_VALUE" "10k 1%"
 			(at 89.662 106.426 0)
+			(show_name no)
+			(do_not_autoplace no)
+			(effects
+				(font
+					(size 1.27 1.27)
+				)
+				(justify right bottom)
+			)
+		)
+		(property "JLCPCB Part #" "C17902"
+			(at 89.662 106.426 0)
+			(hide yes)
+			(show_name no)
+			(do_not_autoplace no)
+			(effects
+				(font
+					(size 1.27 1.27)
+				)
+				(justify right bottom)
+			)
+		)
+		(property "Manufacturer" "UNI-ROYAL"
+			(at 89.662 106.426 0)
+			(hide yes)
+			(show_name no)
+			(do_not_autoplace no)
+			(effects
+				(font
+					(size 1.27 1.27)
+				)
+				(justify right bottom)
+			)
+		)
+		(property "Manufacturer Part #" "1206W4F1002T5E"
+			(at 89.662 106.426 0)
+			(hide yes)
 			(show_name no)
 			(do_not_autoplace no)
@@
 			(project "Trackpoint"
 				(path "/f80cdd06-fe18-4f08-ad78-5d64af2b92b5/a056f087-e621-494b-bb8a-f53c663bfa45"
-					(reference "Ra1")
+					(reference "USB.Ra.1")
 					(unit 4)
 				)
@@
 		(in_pos_files yes)
 		(dnp no)
-		(property "Reference" "Ra1"
+		(property "Reference" "USB.Ra.1"
 			(at 74.422 101.346 0)
 			(show_name no)
@@
 		(property "ALTIUM_VALUE" "10k 1%"
 			(at 74.422 106.426 0)
+			(show_name no)
+			(do_not_autoplace no)
+			(effects
+				(font
+					(size 1.27 1.27)
+				)
+				(justify right bottom)
+			)
+		)
+		(property "JLCPCB Part #" "C17902"
+			(at 74.422 106.426 0)
+			(hide yes)
+			(show_name no)
+			(do_not_autoplace no)
+			(effects
+				(font
+					(size 1.27 1.27)
+				)
+				(justify right bottom)
+			)
+		)
+		(property "Manufacturer" "UNI-ROYAL"
+			(at 74.422 106.426 0)
+			(hide yes)
+			(show_name no)
+			(do_not_autoplace no)
+			(effects
+				(font
+					(size 1.27 1.27)
+				)
+				(justify right bottom)
+			)
+		)
+		(property "Manufacturer Part #" "1206W4F1002T5E"
+			(at 74.422 106.426 0)
+			(hide yes)
 			(show_name no)
 			(do_not_autoplace no)
@@
 			(project "Trackpoint"
 				(path "/f80cdd06-fe18-4f08-ad78-5d64af2b92b5/a056f087-e621-494b-bb8a-f53c663bfa45"
-					(reference "Ra1")
+					(reference "USB.Ra.1")
 					(unit 3)
 				)
@@
 		(in_pos_files yes)
 		(dnp no)
-		(property "Reference" "R7"
+		(property "Reference" "USB.R.7"
 			(at 235.966 100.838 90)
 			(show_name no)
@@
 			(project "Trackpoint"
 				(path "/f80cdd06-fe18-4f08-ad78-5d64af2b92b5/a056f087-e621-494b-bb8a-f53c663bfa45"
-					(reference "R7")
+					(reference "USB.R.7")
 					(unit 1)
 				)
@@
 		(in_pos_files yes)
 		(dnp no)
-		(property "Reference" "FB3"
+		(property "Reference" "USB.FB.3"
 			(at 198.12 101.6 90)
 			(show_name no)
@@
 			(project "Trackpoint"
 				(path "/f80cdd06-fe18-4f08-ad78-5d64af2b92b5/a056f087-e621-494b-bb8a-f53c663bfa45"
-					(reference "FB3")
+					(reference "USB.FB.3")
 					(unit 1)
 				)
@@
 		(in_pos_files yes)
 		(dnp no)
-		(property "Reference" "Z1"
+		(property "Reference" "USB.Z.1"
 			(at 177.8 134.62 90)
 			(show_name no)
@@
 			(project "Trackpoint"
 				(path "/f80cdd06-fe18-4f08-ad78-5d64af2b92b5/a056f087-e621-494b-bb8a-f53c663bfa45"
-					(reference "Z1")
+					(reference "USB.Z.1")
 					(unit 1)
 				)
@@
 		(in_pos_files yes)
 		(dnp no)
-		(property "Reference" "R6"
+		(property "Reference" "USB.R.6"
 			(at 235.966 90.678 90)
 			(show_name no)
@@
 			(project "Trackpoint"
 				(path "/f80cdd06-fe18-4f08-ad78-5d64af2b92b5/a056f087-e621-494b-bb8a-f53c663bfa45"
-					(reference "R6")
+					(reference "USB.R.6")
 					(unit 1)
 				)
@@
 		(in_pos_files yes)
 		(dnp no)
-		(property "Reference" "J3"
+		(property "Reference" "USB.J.3"
 			(at 20.32 63.5 90)
 			(show_name no)
@@
 			(project "Trackpoint"
 				(path "/f80cdd06-fe18-4f08-ad78-5d64af2b92b5/a056f087-e621-494b-bb8a-f53c663bfa45"
-					(reference "J3")
+					(reference "USB.J.3")
 					(unit 1)
 				)
@@
 		(in_pos_files yes)
 		(dnp no)
-		(property "Reference" "FB1"
+		(property "Reference" "USB.FB.1"
 			(at 198.12 71.12 90)
 			(show_name no)
@@
 			(project "Trackpoint"
 				(path "/f80cdd06-fe18-4f08-ad78-5d64af2b92b5/a056f087-e621-494b-bb8a-f53c663bfa45"
-					(reference "FB1")
+					(reference "USB.FB.1")
 					(unit 1)
 				)
@@
 		(in_pos_files yes)
 		(dnp no)
-		(property "Reference" "Ra1"
+		(property "Reference" "USB.Ra.1"
 			(at 107.442 101.346 0)
 			(show_name no)
@@
 		(property "ALTIUM_VALUE" "10k 1%"
 			(at 107.442 106.426 0)
+			(show_name no)
+			(do_not_autoplace no)
+			(effects
+				(font
+					(size 1.27 1.27)
+				)
+				(justify right bottom)
+			)
+		)
+		(property "JLCPCB Part #" "C17902"
+			(at 107.442 106.426 0)
+			(hide yes)
+			(show_name no)
+			(do_not_autoplace no)
+			(effects
+				(font
+					(size 1.27 1.27)
+				)
+				(justify right bottom)
+			)
+		)
+		(property "Manufacturer" "UNI-ROYAL"
+			(at 107.442 106.426 0)
+			(hide yes)
+			(show_name no)
+			(do_not_autoplace no)
+			(effects
+				(font
+					(size 1.27 1.27)
+				)
+				(justify right bottom)
+			)
+		)
+		(property "Manufacturer Part #" "1206W4F1002T5E"
+			(at 107.442 106.426 0)
+			(hide yes)
 			(show_name no)
 			(do_not_autoplace no)
@@
 			(project "Trackpoint"
 				(path "/f80cdd06-fe18-4f08-ad78-5d64af2b92b5/a056f087-e621-494b-bb8a-f53c663bfa45"
-					(reference "Ra1")
+					(reference "USB.Ra.1")
 					(unit 1)
 				)
