File: hardware/electronics/PCBs/Trackpoint_KiCad/MCU.kicad_sch (KiCad schematic)
At the start: 16 parts, among them J1 HEADER2, U1 W25Q16JVSSIQ, U5 RP2040, Y1 RH100-12.000-16-3030

Commit message: Update all components to jlcpcb compatible
Parts:
- MCU.U.1: renamed from U1; JLCPCB Part # (none) -> C82317; Manufacturer (none) -> Winbond Elec
- renumbered C1 to MCU.C.1, C2 to MCU.C.2, C21 to MCU.C.21, C22 to MCU.C.22, C3 to MCU.C.3, C4 to MCU.C.4, C5 to MCU.C.5, C6 to MCU.C.6, C7 to MCU.C.7, J1 to MCU.J.1, R1 to MCU.R.1, R11 to MCU.R.11, R2 to MCU.R.2, U5 to MCU.U.5, Y1 to MCU.Y.1
Changed lines of the file:
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@@
 		(in_pos_files yes)
 		(dnp no)
-		(property "Reference" "C1"
+		(property "Reference" "MCU.C.1"
 			(at 286.766 98.6282 0)
 			(show_name no)
@@
 			(project "Trackpoint"
 				(path "/f80cdd06-fe18-4f08-ad78-5d64af2b92b5/61e63e2a-679d-4322-b593-e2d34443bebf"
-					(reference "C1")
+					(reference "MCU.C.1")
 					(unit 1)
 				)
@@
 		(in_pos_files yes)
 		(dnp no)
-		(property "Reference" "C22"
+		(property "Reference" "MCU.C.22"
 			(at 261.366 207.8482 0)
 			(show_name no)
@@
 			(project "Trackpoint"
 				(path "/f80cdd06-fe18-4f08-ad78-5d64af2b92b5/61e63e2a-679d-4322-b593-e2d34443bebf"
-					(reference "C22")
+					(reference "MCU.C.22")
 					(unit 1)
 				)
@@
 		(in_pos_files yes)
 		(dnp no)
-		(property "Reference" "J1"
+		(property "Reference" "MCU.J.1"
 			(at 175.26 76.0222 90)
 			(show_name no)
@@
 			(project "Trackpoint"
 				(path "/f80cdd06-fe18-4f08-ad78-5d64af2b92b5/61e63e2a-679d-4322-b593-e2d34443bebf"
-					(reference "J1")
+					(reference "MCU.J.1")
 					(unit 1)
 				)
@@
 		(in_pos_files yes)
 		(dnp no)
-		(property "Reference" "C3"
+		(property "Reference" "MCU.C.3"
 			(at 340.106 146.8882 0)
 			(show_name no)
@@
 			(project "Trackpoint"
 				(path "/f80cdd06-fe18-4f08-ad78-5d64af2b92b5/61e63e2a-679d-4322-b593-e2d34443bebf"
-					(reference "C3")
+					(reference "MCU.C.3")
 					(unit 1)
 				)
@@
 		(in_pos_files yes)
 		(dnp no)
-		(property "Reference" "U1"
+		(property "Reference" "MCU.U.1"
 			(at 231.14 91.2622 90)
 			(show_name no)
@@
 		)
 		(property "SUPPLIER PART NUMBER 1" "W25Q16JVSSIQ-ND"
+			(at 212.852 37.9222 90)
+			(hide yes)
+			(show_name no)
+			(do_not_autoplace no)
+			(effects
+				(font
+					(size 1.27 1.27)
+				)
+				(justify right bottom)
+			)
+		)
+		(property "JLCPCB Part #" "C82317"
+			(at 212.852 37.9222 90)
+			(hide yes)
+			(show_name no)
+			(do_not_autoplace no)
+			(effects
+				(font
+					(size 1.27 1.27)
+				)
+				(justify right bottom)
+			)
+		)
+		(property "Manufacturer" "Winbond Elec"
 			(at 212.852 37.9222 90)
 			(hide yes)
@@
 			(project "Trackpoint"
 				(path "/f80cdd06-fe18-4f08-ad78-5d64af2b92b5/61e63e2a-679d-4322-b593-e2d34443bebf"
-					(reference "U1")
+					(reference "MCU.U.1")
 					(unit 1)
 				)
@@
 		(in_pos_files yes)
 		(dnp no)
-		(property "Reference" "R1"
+		(property "Reference" "MCU.R.1"
 			(at 205.486 77.8002 90)
 			(show_name no)
@@
 			(project "Trackpoint"
 				(path "/f80cdd06-fe18-4f08-ad78-5d64af2b92b5/61e63e2a-679d-4322-b593-e2d34443bebf"
-					(reference "R1")
+					(reference "MCU.R.1")
 					(unit 1)
 				)
@@
 		(in_pos_files yes)
 		(dnp no)
-		(property "Reference" "C5"
+		(property "Reference" "MCU.C.5"
 			(at 304.546 159.5882 0)
 			(show_name no)
@@
 			(project "Trackpoint"
 				(path "/f80cdd06-fe18-4f08-ad78-5d64af2b92b5/61e63e2a-679d-4322-b593-e2d34443bebf"
-					(reference "C5")
+					(reference "MCU.C.5")
 					(unit 1)
 				)
@@
 		(in_pos_files yes)
 		(dnp no)
-		(property "Reference" "C6"
+		(property "Reference" "MCU.C.6"
 			(at 286.766 164.6682 0)
 			(show_name no)
@@
 			(project "Trackpoint"
 				(path "/f80cdd06-fe18-4f08-ad78-5d64af2b92b5/61e63e2a-679d-4322-b593-e2d34443bebf"
-					(reference "C6")
+					(reference "MCU.C.6")
 					(unit 1)
 				)
@@
 		(in_pos_files yes)
 		(dnp no)
-		(property "Reference" "Y1"
+		(property "Reference" "MCU.Y.1"
 			(at 109.22 192.8622 90)
 			(show_name no)
@@
 			(project "Trackpoint"
 				(path "/f80cdd06-fe18-4f08-ad78-5d64af2b92b5/61e63e2a-679d-4322-b593-e2d34443bebf"
-					(reference "Y1")
+					(reference "MCU.Y.1")
 					(unit 1)
 				)
@@
 		(in_pos_files yes)
 		(dnp no)
-		(property "Reference" "U5"
+		(property "Reference" "MCU.U.5"
 			(at 154.94 93.8022 90)
 			(show_name no)
@@
 			(project "Trackpoint"
 				(path "/f80cdd06-fe18-4f08-ad78-5d64af2b92b5/61e63e2a-679d-4322-b593-e2d34443bebf"
-					(reference "U5")
+					(reference "MCU.U.5")
 					(unit 1)
 				)
@@
 		(in_pos_files yes)
 		(dnp no)
-		(property "Reference" "R2"
+		(property "Reference" "MCU.R.2"
 			(at 230.886 77.8002 90)
 			(show_name no)
@@
 			(project "Trackpoint"
 				(path "/f80cdd06-fe18-4f08-ad78-5d64af2b92b5/61e63e2a-679d-4322-b593-e2d34443bebf"
-					(reference "R2")
+					(reference "MCU.R.2")
 					(unit 1)
 				)
@@
 		(in_pos_files yes)
 		(dnp no)
-		(property "Reference" "C2"
+		(property "Reference" "MCU.C.2"
 			(at 360.426 139.2682 0)
 			(show_name no)
@@
 			(project "Trackpoint"
 				(path "/f80cdd06-fe18-4f08-ad78-5d64af2b92b5/61e63e2a-679d-4322-b593-e2d34443bebf"
-					(reference "C2")
+					(reference "MCU.C.2")
 					(unit 1)
 				)
@@
 		(in_pos_files yes)
 		(dnp no)
-		(property "Reference" "C4"
+		(property "Reference" "MCU.C.4"
 			(at 322.326 151.9682 0)
 			(show_name no)
@@
 			(project "Trackpoint"
 				(path "/f80cdd06-fe18-4f08-ad78-5d64af2b92b5/61e63e2a-679d-4322-b593-e2d34443bebf"
-					(reference "C4")
+					(reference "MCU.C.4")
 					(unit 1)
 				)
@@
 		(in_pos_files yes)
 		(dnp no)
-		(property "Reference" "R11"
+		(property "Reference" "MCU.R.11"
 			(at 124.206 199.7202 90)
 			(show_name no)
@@
 			(project "Trackpoint"
 				(path "/f80cdd06-fe18-4f08-ad78-5d64af2b92b5/61e63e2a-679d-4322-b593-e2d34443bebf"
-					(reference "R11")
+					(reference "MCU.R.11")
 					(unit 1)
 				)
@@
 		(in_pos_files yes)
 		(dnp no)
-		(property "Reference" "C7"
+		(property "Reference" "MCU.C.7"
 			(at 251.206 177.3682 0)
 			(show_name no)
@@
 			(project "Trackpoint"
 				(path "/f80cdd06-fe18-4f08-ad78-5d64af2b92b5/61e63e2a-679d-4322-b593-e2d34443bebf"
-					(reference "C7")
+					(reference "MCU.C.7")
 					(unit 1)
 				)
@@
 		(in_pos_files yes)
 		(dnp no)
-		(property "Reference" "C21"
+		(property "Reference" "MCU.C.21"
 			(at 279.146 200.2282 0)
 			(show_name no)
@@
 			(project "Trackpoint"
 				(path "/f80cdd06-fe18-4f08-ad78-5d64af2b92b5/61e63e2a-679d-4322-b593-e2d34443bebf"
-					(reference "C21")
+					(reference "MCU.C.21")
 					(unit 1)
 				)
