File: hardware/electronics/PCBs/Trackpoint_KiCad/Mechanical.kicad_sch (KiCad schematic)
At the start: 27 parts

Commit message: Update all components to jlcpcb compatible
Parts:
- renumbered FID1 to MCH.FID.1, FID2 to MCH.FID.2, FID3 to MCH.FID.3, FID4 to MCH.FID.4, FID5 to MCH.FID.5, FID6 to MCH.FID.6, LOGO2 to MCH.LOGO.2, SP1 to MCH.SP.1, SP10 to MCH.SP.10, SP11 to MCH.SP.11, SP12 to MCH.SP.12, SP13 to MCH.SP.13, SP14 to MCH.SP.14, SP15 to MCH.SP.15, SP16 to MCH.SP.16, SP17 to MCH.SP.17, SP18 to MCH.SP.18, SP19 to MCH.SP.19, SP2 to MCH.SP.2, SP20 to MCH.SP.20, SP3 to MCH.SP.3, SP4 to MCH.SP.4, SP5 to MCH.SP.5, SP6 to MCH.SP.6, SP7 to MCH.SP.7, SP8 to MCH.SP.8, SP9 to MCH.SP.9
Changed lines of the file:
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@@
 		(in_pos_files yes)
 		(dnp no)
-		(property "Reference" "SP3"
+		(property "Reference" "MCH.SP.3"
 			(at 185.42 88.9 90)
 			(show_name no)
@@
 			(project "Trackpoint"
 				(path "/f80cdd06-fe18-4f08-ad78-5d64af2b92b5/0a470cbc-6b38-46b7-9538-751fb8c3ae56"
-					(reference "SP3")
+					(reference "MCH.SP.3")
 					(unit 1)
 				)
@@
 		(in_pos_files yes)
 		(dnp no)
-		(property "Reference" "SP8"
+		(property "Reference" "MCH.SP.8"
 			(at 176.53 93.98 90)
 			(show_name no)
@@
 			(project "Trackpoint"
 				(path "/f80cdd06-fe18-4f08-ad78-5d64af2b92b5/0a470cbc-6b38-46b7-9538-751fb8c3ae56"
-					(reference "SP8")
+					(reference "MCH.SP.8")
 					(unit 1)
 				)
@@
 		(in_pos_files yes)
 		(dnp no)
-		(property "Reference" "FID2"
+		(property "Reference" "MCH.FID.2"
 			(at 85.09 71.12 90)
 			(show_name no)
@@
 			(project "Trackpoint"
 				(path "/f80cdd06-fe18-4f08-ad78-5d64af2b92b5/0a470cbc-6b38-46b7-9538-751fb8c3ae56"
-					(reference "FID2")
+					(reference "MCH.FID.2")
 					(unit 1)
 				)
@@
 		(in_pos_files yes)
 		(dnp no)
-		(property "Reference" "LOGO2"
+		(property "Reference" "MCH.LOGO.2"
 			(at 76.2 114.3 90)
 			(show_name no)
@@
 			(project "Trackpoint"
 				(path "/f80cdd06-fe18-4f08-ad78-5d64af2b92b5/0a470cbc-6b38-46b7-9538-751fb8c3ae56"
-					(reference "LOGO2")
+					(reference "MCH.LOGO.2")
 					(unit 1)
 				)
@@
 		(in_pos_files yes)
 		(dnp no)
-		(property "Reference" "SP7"
+		(property "Reference" "MCH.SP.7"
 			(at 170.18 86.36 90)
 			(show_name no)
@@
 			(project "Trackpoint"
 				(path "/f80cdd06-fe18-4f08-ad78-5d64af2b92b5/0a470cbc-6b38-46b7-9538-751fb8c3ae56"
-					(reference "SP7")
+					(reference "MCH.SP.7")
 					(unit 1)
 				)
@@
 		(in_pos_files yes)
 		(dnp no)
-		(property "Reference" "SP1"
+		(property "Reference" "MCH.SP.1"
 			(at 172.72 88.9 90)
 			(show_name no)
@@
 			(project "Trackpoint"
 				(path "/f80cdd06-fe18-4f08-ad78-5d64af2b92b5/0a470cbc-6b38-46b7-9538-751fb8c3ae56"
-					(reference "SP1")
+					(reference "MCH.SP.1")
 					(unit 1)
 				)
@@
 		(in_pos_files yes)
 		(dnp no)
-		(property "Reference" "SP4"
+		(property "Reference" "MCH.SP.4"
 			(at 190.5 91.44 90)
 			(show_name no)
@@
 			(project "Trackpoint"
 				(path "/f80cdd06-fe18-4f08-ad78-5d64af2b92b5/0a470cbc-6b38-46b7-9538-751fb8c3ae56"
-					(reference "SP4")
+					(reference "MCH.SP.4")
 					(unit 1)
 				)
@@
 		(in_pos_files yes)
 		(dnp no)
-		(property "Reference" "FID5"
+		(property "Reference" "MCH.FID.5"
 			(at 54.61 93.98 90)
 			(show_name no)
@@
 			(project "Trackpoint"
 				(path "/f80cdd06-fe18-4f08-ad78-5d64af2b92b5/0a470cbc-6b38-46b7-9538-751fb8c3ae56"
-					(reference "FID5")
+					(reference "MCH.FID.5")
 					(unit 1)
 				)
@@
 		(in_pos_files yes)
 		(dnp no)
-		(property "Reference" "SP20"
+		(property "Reference" "MCH.SP.20"
 			(at 203.2 119.38 90)
 			(show_name no)
@@
 			(project "Trackpoint"
 				(path "/f80cdd06-fe18-4f08-ad78-5d64af2b92b5/0a470cbc-6b38-46b7-9538-751fb8c3ae56"
-					(reference "SP20")
+					(reference "MCH.SP.20")
 					(unit 1)
 				)
@@
 		(in_pos_files yes)
 		(dnp no)
-		(property "Reference" "SP9"
+		(property "Reference" "MCH.SP.9"
 			(at 182.88 86.36 90)
 			(show_name no)
@@
 			(project "Trackpoint"
 				(path "/f80cdd06-fe18-4f08-ad78-5d64af2b92b5/0a470cbc-6b38-46b7-9538-751fb8c3ae56"
-					(reference "SP9")
+					(reference "MCH.SP.9")
 					(unit 1)
 				)
@@
 		(in_pos_files yes)
 		(dnp no)
-		(property "Reference" "SP11"
+		(property "Reference" "MCH.SP.11"
 			(at 195.58 86.36 90)
 			(show_name no)
@@
 			(project "Trackpoint"
 				(path "/f80cdd06-fe18-4f08-ad78-5d64af2b92b5/0a470cbc-6b38-46b7-9538-751fb8c3ae56"
-					(reference "SP11")
+					(reference "MCH.SP.11")
 					(unit 1)
 				)
@@
 		(in_pos_files yes)
 		(dnp no)
-		(property "Reference" "SP17"
+		(property "Reference" "MCH.SP.17"
 			(at 187.96 111.76 90)
 			(show_name no)
@@
 			(project "Trackpoint"
 				(path "/f80cdd06-fe18-4f08-ad78-5d64af2b92b5/0a470cbc-6b38-46b7-9538-751fb8c3ae56"
-					(reference "SP17")
+					(reference "MCH.SP.17")
 					(unit 1)
 				)
@@
 		(in_pos_files yes)
 		(dnp no)
-		(property "Reference" "FID1"
+		(property "Reference" "MCH.FID.1"
 			(at 54.61 71.12 90)
 			(show_name no)
@@
 			(project "Trackpoint"
 				(path "/f80cdd06-fe18-4f08-ad78-5d64af2b92b5/0a470cbc-6b38-46b7-9538-751fb8c3ae56"
-					(reference "FID1")
+					(reference "MCH.FID.1")
 					(unit 1)
 				)
@@
 		(in_pos_files yes)
 		(dnp no)
-		(property "Reference" "SP15"
+		(property "Reference" "MCH.SP.15"
 			(at 177.8 116.84 90)
 			(show_name no)
@@
 			(project "Trackpoint"
 				(path "/f80cdd06-fe18-4f08-ad78-5d64af2b92b5/0a470cbc-6b38-46b7-9538-751fb8c3ae56"
-					(reference "SP15")
+					(reference "MCH.SP.15")
 					(unit 1)
 				)
@@
 		(in_pos_files yes)
 		(dnp no)
-		(property "Reference" "SP13"
+		(property "Reference" "MCH.SP.13"
 			(at 170.18 111.76 90)
 			(show_name no)
@@
 			(project "Trackpoint"
 				(path "/f80cdd06-fe18-4f08-ad78-5d64af2b92b5/0a470cbc-6b38-46b7-9538-751fb8c3ae56"
-					(reference "SP13")
+					(reference "MCH.SP.13")
 					(unit 1)
 				)
@@
 		(in_pos_files yes)
 		(dnp no)
-		(property "Reference" "SP19"
+		(property "Reference" "MCH.SP.19"
 			(at 198.12 116.84 90)
 			(show_name no)
@@
 			(project "Trackpoint"
 				(path "/f80cdd06-fe18-4f08-ad78-5d64af2b92b5/0a470cbc-6b38-46b7-9538-751fb8c3ae56"
-					(reference "SP19")
+					(reference "MCH.SP.19")
 					(unit 1)
 				)
@@
 		(in_pos_files yes)
 		(dnp no)
-		(property "Reference" "SP14"
+		(property "Reference" "MCH.SP.14"
 			(at 172.72 114.3 90)
 			(show_name no)
@@
 			(project "Trackpoint"
 				(path "/f80cdd06-fe18-4f08-ad78-5d64af2b92b5/0a470cbc-6b38-46b7-9538-751fb8c3ae56"
-					(reference "SP14")
+					(reference "MCH.SP.14")
 					(unit 1)
 				)
@@
 		(in_pos_files yes)
 		(dnp no)
-		(property "Reference" "SP2"
+		(property "Reference" "MCH.SP.2"
 			(at 177.8 91.44 90)
 			(show_name no)
@@
 			(project "Trackpoint"
 				(path "/f80cdd06-fe18-4f08-ad78-5d64af2b92b5/0a470cbc-6b38-46b7-9538-751fb8c3ae56"
-					(reference "SP2")
+					(reference "MCH.SP.2")
 					(unit 1)
 				)
@@
 		(in_pos_files yes)
 		(dnp no)
-		(property "Reference" "SP16"
+		(property "Reference" "MCH.SP.16"
 			(at 182.88 119.38 90)
 			(show_name no)
@@
 			(project "Trackpoint"
 				(path "/f80cdd06-fe18-4f08-ad78-5d64af2b92b5/0a470cbc-6b38-46b7-9538-751fb8c3ae56"
-					(reference "SP16")
+					(reference "MCH.SP.16")
 					(unit 1)
 				)
@@
 		(in_pos_files yes)
 		(dnp no)
-		(property "Reference" "SP10"
+		(property "Reference" "MCH.SP.10"
 			(at 189.23 93.98 90)
 			(show_name no)
@@
 			(project "Trackpoint"
 				(path "/f80cdd06-fe18-4f08-ad78-5d64af2b92b5/0a470cbc-6b38-46b7-9538-751fb8c3ae56"
-					(reference "SP10")
+					(reference "MCH.SP.10")
 					(unit 1)
 				)
@@
 		(in_pos_files yes)
 		(dnp no)
-		(property "Reference" "SP12"
+		(property "Reference" "MCH.SP.12"
 			(at 201.93 93.98 90)
 			(show_name no)
@@
 			(project "Trackpoint"
 				(path "/f80cdd06-fe18-4f08-ad78-5d64af2b92b5/0a470cbc-6b38-46b7-9538-751fb8c3ae56"
-					(reference "SP12")
+					(reference "MCH.SP.12")
 					(unit 1)
 				)
@@
 		(in_pos_files yes)
 		(dnp no)
-		(property "Reference" "SP18"
+		(property "Reference" "MCH.SP.18"
 			(at 193.04 114.3 90)
 			(show_name no)
@@
 			(project "Trackpoint"
 				(path "/f80cdd06-fe18-4f08-ad78-5d64af2b92b5/0a470cbc-6b38-46b7-9538-751fb8c3ae56"
-					(reference "SP18")
+					(reference "MCH.SP.18")
 					(unit 1)
 				)
@@
 		(in_pos_files yes)
 		(dnp no)
-		(property "Reference" "FID4"
+		(property "Reference" "MCH.FID.4"
 			(at 85.09 82.55 90)
 			(show_name no)
@@
 			(project "Trackpoint"
 				(path "/f80cdd06-fe18-4f08-ad78-5d64af2b92b5/0a470cbc-6b38-46b7-9538-751fb8c3ae56"
-					(reference "FID4")
+					(reference "MCH.FID.4")
 					(unit 1)
 				)
@@
 		(in_pos_files yes)
 		(dnp no)
-		(property "Reference" "FID6"
+		(property "Reference" "MCH.FID.6"
 			(at 85.09 93.98 90)
 			(show_name no)
@@
 			(project "Trackpoint"
 				(path "/f80cdd06-fe18-4f08-ad78-5d64af2b92b5/0a470cbc-6b38-46b7-9538-751fb8c3ae56"
-					(reference "FID6")
+					(reference "MCH.FID.6")
 					(unit 1)
 				)
@@
 		(in_pos_files yes)
 		(dnp no)
-		(property "Reference" "SP5"
+		(property "Reference" "MCH.SP.5"
 			(at 198.12 88.9 90)
 			(show_name no)
@@
 			(project "Trackpoint"
 				(path "/f80cdd06-fe18-4f08-ad78-5d64af2b92b5/0a470cbc-6b38-46b7-9538-751fb8c3ae56"
-					(reference "SP5")
+					(reference "MCH.SP.5")
 					(unit 1)
 				)
@@
 		(in_pos_files yes)
 		(dnp no)
-		(property "Reference" "SP6"
+		(property "Reference" "MCH.SP.6"
 			(at 203.2 91.44 90)
 			(show_name no)
@@
 			(project "Trackpoint"
 				(path "/f80cdd06-fe18-4f08-ad78-5d64af2b92b5/0a470cbc-6b38-46b7-9538-751fb8c3ae56"
-					(reference "SP6")
+					(reference "MCH.SP.6")
 					(unit 1)
 				)
@@
 		(in_pos_files yes)
 		(dnp no)
-		(property "Reference" "FID3"
+		(property "Reference" "MCH.FID.3"
 			(at 54.61 82.55 90)
 			(show_name no)
@@
 			(project "Trackpoint"
 				(path "/f80cdd06-fe18-4f08-ad78-5d64af2b92b5/0a470cbc-6b38-46b7-9538-751fb8c3ae56"
-					(reference "FID3")
+					(reference "MCH.FID.3")
 					(unit 1)
 				)
