File: hardware/electronics/PCBs/Trackpoint_KiCad/Regulators.kicad_sch (KiCad schematic)
At the start: 4 parts, among them U3 AP2202K-3.3

Commit message: Update all components to jlcpcb compatible
Parts:
- renumbered C12 to REG.C.12, C13 to REG.C.13, C14 to REG.C.14, U3 to REG.U.3
Changed lines of the file:
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@@
 		(in_pos_files yes)
 		(dnp no)
-		(property "Reference" "C14"
+		(property "Reference" "REG.C.14"
 			(at 177.546 73.406 0)
 			(show_name no)
@@
 			(project "Trackpoint"
 				(path "/f80cdd06-fe18-4f08-ad78-5d64af2b92b5/b283ed3a-f471-4bf8-bb22-476d14500d3a"
-					(reference "C14")
+					(reference "REG.C.14")
 					(unit 1)
 				)
@@
 		(in_pos_files yes)
 		(dnp no)
-		(property "Reference" "C13"
+		(property "Reference" "REG.C.13"
 			(at 162.306 73.406 0)
 			(show_name no)
@@
 			(project "Trackpoint"
 				(path "/f80cdd06-fe18-4f08-ad78-5d64af2b92b5/b283ed3a-f471-4bf8-bb22-476d14500d3a"
-					(reference "C13")
+					(reference "REG.C.13")
 					(unit 1)
 				)
@@
 		(in_pos_files yes)
 		(dnp no)
-		(property "Reference" "U3"
+		(property "Reference" "REG.U.3"
 			(at 116.84 66.04 90)
 			(show_name no)
@@
 			(project "Trackpoint"
 				(path "/f80cdd06-fe18-4f08-ad78-5d64af2b92b5/b283ed3a-f471-4bf8-bb22-476d14500d3a"
-					(reference "U3")
+					(reference "REG.U.3")
 					(unit 1)
 				)
@@
 		(in_pos_files yes)
 		(dnp no)
-		(property "Reference" "C12"
+		(property "Reference" "REG.C.12"
 			(at 101.346 73.406 0)
 			(show_name no)
@@
 			(project "Trackpoint"
 				(path "/f80cdd06-fe18-4f08-ad78-5d64af2b92b5/b283ed3a-f471-4bf8-bb22-476d14500d3a"
-					(reference "C12")
+					(reference "REG.C.12")
 					(unit 1)
 				)
