File: hardware/electronics/PCBs/Trackpoint_KiCad/RotSense.kicad_sch (KiCad schematic)
At the start: 3 parts, among them U6 TMAG5273

Commit message: Update all components to jlcpcb compatible
Parts:
- RSN.Ra.2: renamed from Ra2; JLCPCB Part # (none) -> C52199; Manufacturer (none) -> UNI-ROYAL; Manufacturer Part # (none) -> 1206W4F1001T5E
- renumbered C9 to RSN.C.9, U6 to RSN.U.6
Changed lines of the file:
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@@
 		(in_pos_files yes)
 		(dnp no)
-		(property "Reference" "Ra2"
+		(property "Reference" "RSN.Ra.2"
 			(at 115.062 83.566 0)
 			(show_name no)
@@
 		(property "ALTIUM_VALUE" "1k 1%"
 			(at 115.062 88.646 0)
+			(show_name no)
+			(do_not_autoplace no)
+			(effects
+				(font
+					(size 1.27 1.27)
+				)
+				(justify right bottom)
+			)
+		)
+		(property "JLCPCB Part #" "C52199"
+			(at 115.062 88.646 0)
+			(hide yes)
+			(show_name no)
+			(do_not_autoplace no)
+			(effects
+				(font
+					(size 1.27 1.27)
+				)
+				(justify right bottom)
+			)
+		)
+		(property "Manufacturer" "UNI-ROYAL"
+			(at 115.062 88.646 0)
+			(hide yes)
+			(show_name no)
+			(do_not_autoplace no)
+			(effects
+				(font
+					(size 1.27 1.27)
+				)
+				(justify right bottom)
+			)
+		)
+		(property "Manufacturer Part #" "1206W4F1001T5E"
+			(at 115.062 88.646 0)
+			(hide yes)
 			(show_name no)
 			(do_not_autoplace no)
@@
 			(project "Trackpoint"
 				(path "/f80cdd06-fe18-4f08-ad78-5d64af2b92b5/840bc58a-fb72-4e84-8a46-91a0827a7de5"
-					(reference "Ra2")
+					(reference "RSN.Ra.2")
 					(unit 2)
 				)
@@
 		(in_pos_files yes)
 		(dnp no)
-		(property "Reference" "Ra2"
+		(property "Reference" "RSN.Ra.2"
 			(at 130.302 83.566 0)
 			(show_name no)
@@
 		(property "ALTIUM_VALUE" "1k 1%"
 			(at 130.302 88.646 0)
+			(show_name no)
+			(do_not_autoplace no)
+			(effects
+				(font
+					(size 1.27 1.27)
+				)
+				(justify right bottom)
+			)
+		)
+		(property "JLCPCB Part #" "C52199"
+			(at 130.302 88.646 0)
+			(hide yes)
+			(show_name no)
+			(do_not_autoplace no)
+			(effects
+				(font
+					(size 1.27 1.27)
+				)
+				(justify right bottom)
+			)
+		)
+		(property "Manufacturer" "UNI-ROYAL"
+			(at 130.302 88.646 0)
+			(hide yes)
+			(show_name no)
+			(do_not_autoplace no)
+			(effects
+				(font
+					(size 1.27 1.27)
+				)
+				(justify right bottom)
+			)
+		)
+		(property "Manufacturer Part #" "1206W4F1001T5E"
+			(at 130.302 88.646 0)
+			(hide yes)
 			(show_name no)
 			(do_not_autoplace no)
@@
 			(project "Trackpoint"
 				(path "/f80cdd06-fe18-4f08-ad78-5d64af2b92b5/840bc58a-fb72-4e84-8a46-91a0827a7de5"
-					(reference "Ra2")
+					(reference "RSN.Ra.2")
 					(unit 4)
 				)
@@
 		(in_pos_files yes)
 		(dnp no)
-		(property "Reference" "Ra2"
+		(property "Reference" "RSN.Ra.2"
 			(at 130.302 93.726 0)
 			(show_name no)
@@
 		(property "ALTIUM_VALUE" "1k 1%"
 			(at 130.302 98.806 0)
+			(show_name no)
+			(do_not_autoplace no)
+			(effects
+				(font
+					(size 1.27 1.27)
+				)
+				(justify right bottom)
+			)
+		)
+		(property "JLCPCB Part #" "C52199"
+			(at 130.302 98.806 0)
+			(hide yes)
+			(show_name no)
+			(do_not_autoplace no)
+			(effects
+				(font
+					(size 1.27 1.27)
+				)
+				(justify right bottom)
+			)
+		)
+		(property "Manufacturer" "UNI-ROYAL"
+			(at 130.302 98.806 0)
+			(hide yes)
+			(show_name no)
+			(do_not_autoplace no)
+			(effects
+				(font
+					(size 1.27 1.27)
+				)
+				(justify right bottom)
+			)
+		)
+		(property "Manufacturer Part #" "1206W4F1001T5E"
+			(at 130.302 98.806 0)
+			(hide yes)
 			(show_name no)
 			(do_not_autoplace no)
@@
 			(project "Trackpoint"
 				(path "/f80cdd06-fe18-4f08-ad78-5d64af2b92b5/840bc58a-fb72-4e84-8a46-91a0827a7de5"
-					(reference "Ra2")
+					(reference "RSN.Ra.2")
 					(unit 3)
 				)
@@
 		(in_pos_files yes)
 		(dnp no)
-		(property "Reference" "Ra2"
+		(property "Reference" "RSN.Ra.2"
 			(at 115.062 93.726 0)
 			(show_name no)
@@
 		(property "ALTIUM_VALUE" "1k 1%"
 			(at 115.062 98.806 0)
+			(show_name no)
+			(do_not_autoplace no)
+			(effects
+				(font
+					(size 1.27 1.27)
+				)
+				(justify right bottom)
+			)
+		)
+		(property "JLCPCB Part #" "C52199"
+			(at 115.062 98.806 0)
+			(hide yes)
+			(show_name no)
+			(do_not_autoplace no)
+			(effects
+				(font
+					(size 1.27 1.27)
+				)
+				(justify right bottom)
+			)
+		)
+		(property "Manufacturer" "UNI-ROYAL"
+			(at 115.062 98.806 0)
+			(hide yes)
+			(show_name no)
+			(do_not_autoplace no)
+			(effects
+				(font
+					(size 1.27 1.27)
+				)
+				(justify right bottom)
+			)
+		)
+		(property "Manufacturer Part #" "1206W4F1001T5E"
+			(at 115.062 98.806 0)
+			(hide yes)
 			(show_name no)
 			(do_not_autoplace no)
@@
 			(project "Trackpoint"
 				(path "/f80cdd06-fe18-4f08-ad78-5d64af2b92b5/840bc58a-fb72-4e84-8a46-91a0827a7de5"
-					(reference "Ra2")
+					(reference "RSN.Ra.2")
 					(unit 1)
 				)
@@
 		(in_pos_files yes)
 		(dnp no)
-		(property "Reference" "C9"
+		(property "Reference" "RSN.C.9"
 			(at 197.866 119.126 0)
 			(show_name no)
@@
 			(project "Trackpoint"
 				(path "/f80cdd06-fe18-4f08-ad78-5d64af2b92b5/840bc58a-fb72-4e84-8a46-91a0827a7de5"
-					(reference "C9")
+					(reference "RSN.C.9")
 					(unit 1)
 				)
@@
 		(in_pos_files yes)
 		(dnp no)
-		(property "Reference" "U6"
+		(property "Reference" "RSN.U.6"
 			(at 147.32 111.76 90)
 			(show_name no)
@@
 			(project "Trackpoint"
 				(path "/f80cdd06-fe18-4f08-ad78-5d64af2b92b5/840bc58a-fb72-4e84-8a46-91a0827a7de5"
-					(reference "U6")
+					(reference "RSN.U.6")
 					(unit 1)
 				)
